File: Alchitry_Au/Alchitry_Au.sch (KiCad schematic (older format))
At the start: 8 parts

Commit message: Correcting Alchitry grid and conns
Adding 5V and 3V3 connections as well as a few missing GND lines
Connections:
- net labels added: +3.3V, +5V
- wire segments 54 -> 146
Other:
- moved on the sheet: B1, B2
